File: quantizer2/hardware_design/pcb/quantizer2_v10.brd (EAGLE design)
At the start: 30 x 107.3 mm, 44 parts, among them IC2 LM4040C10IDBZR, IC3 LM1117DT-3.3_NOPB, IC5 MCP4921T-E_MS, IC7 MCP3204-CI_ST, IC9 TL072CD, U1 LM4040C25IDBZR, Y1 8MHz

Commit message: design for fet overdrive and quantizer 2 code updates
Parts:
- C6: value 47pF -> 100pF
Changed lines of the file:
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@@
 <attribute name="PROD_ID" value=" " x="22" y="19" size="1.778" layer="28" rot="MR180" display="off"/>
 </element>
-<element name="C6" library="SparkFun-Capacitors" library_urn="urn:adsk.eagle:library:510" package="0603" package3d_urn="urn:adsk.eagle:package:37414/1" value="47pF" x="27" y="16" smashed="yes" rot="MR0">
+<element name="C6" library="SparkFun-Capacitors" library_urn="urn:adsk.eagle:library:510" package="0603" package3d_urn="urn:adsk.eagle:package:37414/1" value="100pF" x="27" y="16" smashed="yes" rot="MR0">
 <attribute name="NAME" x="27" y="16.762" size="0.6096" layer="26" font="vector" ratio="20" rot="MR0" align="bottom-center"/>
 <attribute name="PROD_ID" value="CAP-00810" x="27" y="16" size="1.778" layer="28" rot="MR0" display="off"/>
