File: quantizer2/hardware_design/pcb/quantizer2_v50.brd (EAGLE design)
At the start: 30 x 107.3 mm, 54 parts, among them IC2 LM4040C10IDBZR, IC3 LM1117DT-3.3_NOPB, IC4 MCP3201-CI_MS, IC5 MCP4921T-E_MS, IC9 TL072CD, U1 LM4040C25IDBZR, Y1 8MHz

Commit message: progress on audio DAC. switched to f446xx for now
Connections:
- net GND: now also QUANTIZEDSIGNAL.P2, SIGNALIN.P2
Changed lines of the file:
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@@
 <via x="21.4" y="82.1" extent="1-16" drill="0.35"/>
 <via x="5.4" y="94.1" extent="1-16" drill="0.35"/>
+<contactref element="SIGNALIN" pad="P2"/>
+<contactref element="QUANTIZEDSIGNAL" pad="P2"/>
 </signal>
 <signal name="VCC">
