File: fet_overdrive/hardware_design/pcb/fet_overdrive_v40.brd (EAGLE design)
At the start: 30 x 107.3 mm, 38 parts, among them IC1 TL072CD, J1 PJ301_THONKICONN6, J2 PJ301_THONKICONN6, Q1 MMBFJ111, Q2 SMMBT3904LT1G

Commit message: changed 1uF to 10uF to keep more low end in audio signal
Parts:
- C13, C14, C16: value 1.0uF -> 10.0uF
Changed lines of the file:
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@@
 <attribute name="VALUE" x="24.384" y="19.05" size="0.6096" layer="28" font="vector" ratio="20" rot="MR0" align="top-center"/>
 </element>
-<element name="C13" library="SparkFun-Capacitors" library_urn="urn:adsk.eagle:library:510" package="0603" package3d_urn="urn:adsk.eagle:package:37414/1" value="1.0uF" x="12.7" y="55.88" smashed="yes" rot="MR0">
+<element name="C13" library="SparkFun-Capacitors" library_urn="urn:adsk.eagle:library:510" package="0603" package3d_urn="urn:adsk.eagle:package:37414/1" value="10.0uF" x="12.7" y="55.88" smashed="yes" rot="MR0">
 <attribute name="NAME" x="12.7" y="56.642" size="0.6096" layer="26" font="vector" ratio="20" rot="MR0" align="bottom-center"/>
 <attribute name="PROD_ID" value="CAP-00868" x="12.7" y="55.88" size="1.778" layer="28" rot="MR0" display="off"/>
@@
 <attribute name="VALUE" x="12.7" y="51.562" size="0.6096" layer="28" font="vector" ratio="20" rot="MR0" align="top-center"/>
 </element>
-<element name="C14" library="SparkFun-Capacitors" library_urn="urn:adsk.eagle:library:510" package="0603" package3d_urn="urn:adsk.eagle:package:37414/1" value="1.0uF" x="24.384" y="16.764" smashed="yes" rot="MR0">
+<element name="C14" library="SparkFun-Capacitors" library_urn="urn:adsk.eagle:library:510" package="0603" package3d_urn="urn:adsk.eagle:package:37414/1" value="10.0uF" x="24.384" y="16.764" smashed="yes" rot="MR0">
 <attribute name="NAME" x="24.384" y="17.526" size="0.6096" layer="26" font="vector" ratio="20" rot="MR0" align="bottom-center"/>
 <attribute name="PROD_ID" value="CAP-00868" x="24.384" y="16.764" size="1.778" layer="28" rot="MR0" display="off"/>
@@
 <attribute name="VALUE" x="15.086" y="12.314" size="0.6096" layer="28" font="vector" ratio="20" rot="MR0" align="top-center"/>
 </element>
-<element name="C16" library="SparkFun-Capacitors" library_urn="urn:adsk.eagle:library:510" package="0603" package3d_urn="urn:adsk.eagle:package:37414/1" value="1.0uF" x="14.986" y="9.906" smashed="yes" rot="MR0">
+<element name="C16" library="SparkFun-Capacitors" library_urn="urn:adsk.eagle:library:510" package="0603" package3d_urn="urn:adsk.eagle:package:37414/1" value="10.0uF" x="14.986" y="9.906" smashed="yes" rot="MR0">
 <attribute name="NAME" x="14.986" y="10.668" size="0.6096" layer="26" font="vector" ratio="20" rot="MR0" align="bottom-center"/>
 <attribute name="PROD_ID" value="CAP-00868" x="14.986" y="9.906" size="1.778" layer="28" rot="MR0" display="off"/>
