File: fet_overdrive/hardware_design/pcb/fet_overdrive_v50.brd (EAGLE design)
At the start: 30 x 107.3 mm, 32 parts, among them IC1 TL072CD, J1 PJ301_THONKICONN6, J2 PJ301_THONKICONN6, Q1 MMBFJ111, Q2 SMMBT3904LT1G

Commit message: progress on audio DAC. switched to f446xx for now
Connections:
- net GND: now also J1.P2, J2.P2
Changed lines of the file:
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@@
 <via x="11.05" y="47.64" extent="1-16" drill="0.508"/>
 <via x="23.77" y="37.95" extent="1-16" drill="0.508"/>
+<contactref element="J1" pad="P2"/>
+<contactref element="J2" pad="P2"/>
 </signal>
 <signal name="5V">
