File: waves/hardware_design/pcb/zif_breakout.sch (EAGLE design)
At the start: 6 parts, among them J8 F31L-1A7H1-11030

Commit message: trying to get LCD to respond
Connections:
- net N$3: now also J8.5; no longer J8.4
Changed lines of the file:
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@@
 <net name="N$3" class="0">
 <segment>
-<pinref part="J8" gate="G$1" pin="4"/>
-<wire x1="281.94" y1="210.82" x2="302.26" y2="210.82" width="0.1524" layer="91"/>
 <wire x1="302.26" y1="210.82" x2="302.26" y2="208.28" width="0.1524" layer="91"/>
 <pinref part="C17" gate="G$1" pin="1"/>
+<pinref part="J8" gate="G$1" pin="5"/>
+<wire x1="281.94" y1="208.28" x2="299.72" y2="208.28" width="0.1524" layer="91"/>
+<wire x1="299.72" y1="208.28" x2="299.72" y2="210.82" width="0.1524" layer="91"/>
+<wire x1="299.72" y1="210.82" x2="302.26" y2="210.82" width="0.1524" layer="91"/>
 </segment>
 </net>
