File: waves/hardware_design/pcb/zif_breakout_v10.brd (EAGLE design)
At the start: 23.9 x 19.3 mm, 6 parts, among them J8 F31L-1A7H1-11030

Commit message: working on implementing clean morph matrix engine
Changed lines of the file:
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@@
 <contactref element="J8" pad="22"/>
 <contactref element="J8" pad="24"/>
-<wire x1="7.7724" y1="10.3632" x2="7.688" y2="10.33" width="0.1524" layer="1"/>
-<wire x1="8.6868" y1="10.3632" x2="8.688" y2="10.33" width="0.1524" layer="1"/>
-<wire x1="8.6868" y1="10.2108" x2="8.688" y2="10.33" width="0.1524" layer="1"/>
+<wire x1="8.688" y1="10.33" x2="8.6868" y2="10.3632" width="0" layer="19" extent="1-1"/>
+<wire x1="7.688" y1="10.33" x2="7.7724" y2="10.3632" width="0" layer="19" extent="1-1"/>
+<wire x1="8.6868" y1="10.2108" x2="8.688" y2="10.33" width="0" layer="19" extent="1-1"/>
 </signal>
 <signal name="LCD_SCK">
