File: waves/hardware_design/pcb/zif_breakout_v20.sch (EAGLE design)
At the start: 6 parts, among them J8 F31L-1A7H1-11030

Commit message: working on implementing clean morph matrix engine
Connections:
- removed net N$13: C16.1, J8.12
- new net N$1: C16.1, J8.19
- net +3V3: now also J8.10, J8.11, J8.12, J8.13, J8.14, J8.28, J8.4, J8.5; no longer J8.17, J8.18, J8.19, J8.20, J8.21, J8.26, J8.27, J8.3
- net GND: now also J8.15, J8.29; no longer J8.16, J8.2
- net LCD_CMD: now also J8.3; no longer J8.28
- net LCD_CS: now also J8.1; no longer J8.30
- net LCD_DIN: now also J8.7, J8.8, J8.9; no longer J8.22, J8.23, J8.24
- net LCD_RESET: now also J8.2; no longer J8.29
- net LCD_SCK: now also J8.6; no longer J8.25
- net N$12: now also J8.18; no longer J8.13
- net N$3: now also J8.26; no longer J8.5
Other:
- moved on the sheet: J8
